File: flex/flex.kicad_sch (KiCad schematic)
At the start: 81 parts, among them J1 Conn_01x04_Female, J2 Conn_01x05_Female, J3 Conn_01x03_Female, J4 Conn_01x06_Female, J5 Conn_01x03_Female, SW10 SW_Push, SW11 SW_Push, SW12 SW_Push, SW15 SW_Push, SW16 SW_Push, SW17 SW_Push, SW2 SW_Push, SW20 SW_Push, SW21 SW_Push, SW22 SW_Push, SW24 SW_Push, SW25 SW_Push, SW26 SW_Push, SW3 SW_Push, SW4 SW_Push, SW6 SW_Push, SW7 SW_Push, SW8 SW_Push

Commit message: bork
Parts:
- removed D1, D10, D11, D12, D13, D15, D16, D17, D2, D20, D27, D31, D32, D35, D36, D9: D, custom:Diode_TH_SOD123, symbol Device:D
- removed D18, D21, D23, D25, D3, D33, D37, D39, D4, D41, D47, D49, D5, D51, D55, D57, D59: SK6812MINI, libs2:YS-SK6812MINI-E_REVERSE, symbol LED:SK6812MINI
- removed D22, D24, D26, D28, D29, D30, D34, D38, D40, D42, D48, D50, D52, D56, D58, D6, D60: SK6812MINI, libs2:YS-SK6812MINI-E_REVERSE_NO_EDGECUT, symbol LED:SK6812MINI
- removed J2: Conn_01x05_Female, customs:PinHeader_1x05_P2.54mm_Vertical, symbol Connector:Conn_01x05_Female
- removed J3, J5: Conn_01x03_Female, Connector_PinHeader_2.54mm:PinHeader_1x03_P2.54mm_Vertical, symbol Connector:Conn_01x03_Female
- removed J4: Conn_01x06_Female, Connector_PinHeader_2.54mm:PinHeader_1x06_P2.54mm_Vertical, symbol Connector:Conn_01x06_Female
- removed SW10, SW11, SW12, SW15, SW16, SW17, SW2, SW20, SW21, SW22, SW24, SW25, SW26, SW3, SW4, SW6, SW7, SW8: SW_Push, custom:SW_MX_reversible, symbol Switch:SW_Push
- added D10, D12: SK6812MINI, libs2:YS-SK6812MINI-E_REVERSE, symbol LED:SK6812MINI
- added D11, D13: SK6812MINI, libs2:YS-SK6812MINI-E_REVERSE_NO_EDGECUT, symbol LED:SK6812MINI
- added D5: D, custom:Diode_TH_SOD123, symbol Device:D
- added J2: Conn_01x03_Female, Connector_PinHeader_2.54mm:PinHeader_1x03_P2.54mm_Vertical, symbol Connector:Conn_01x03_Female
- added SW14, SW19, SW5: SW_Push, custom:SW_MX_reversible, symbol Switch:SW_Push
- C1, C2: value 1u -> C; footprint Capacitor_SMD:C_1206_3216Metric_Pad1.42x1.75mm_HandSolder -> LED_SMD:LED_1206_3216Metric_Pad1.42x1.75mm_HandSolder
- R1, R2: value 330 -> R
Connections:
- net col3 is gone; now on net col5: D19.1 (K)
- net Din: now also R1.2, R2.2, J2.3 (Pin_3); no longer R1.1, R2.1
- net Gnd: now also D10.2 (VSS), D11.2 (VSS), D12.2 (VSS), D13.2 (VSS), J2.2 (Pin_2)
- net Vcc: now also D10.4 (VDD), D11.4 (VDD), D12.4 (VDD), D13.4 (VDD), J2.1 (Pin_1)
- net col2: now also D5.1 (K)
- net col4: now also D14.1 (K)
- net col5: no longer D14.1 (K)
- net at D7.1 (DOUT), D8.1 (DOUT): now also D10.3 (DIN), D11.3 (DIN)
- net at D19.2 (A): now also SW19.2
- net at D14.2 (A): now also SW14.2
- net at D7.3 (DIN), D8.3 (DIN): now also R1.1, R2.1
- net row5 renamed row1
- net row1: now also SW14.1, SW19.1, SW5.1
- new net: D10.1 (DOUT), D11.1 (DOUT), D12.3 (DIN), D13.3 (DIN)
- new net: D5.2 (A), SW5.2
- no-connect marks 1 -> 2
Other:
- note removed: "MCU connector"
- note removed: "RGB connectors"
